Commit message: stage3

File: description/robot.urdf.xacro (robot description, xacro)
@@ -1,4 +1,5 @@
 <?xml version="1.0"?>
-<robot xmlns:xacro="http://www.ros.org/wiki/xacro"  name="robot">
+<robot xmlns:xacro="http://www.ros.org/wiki/xacro" name="robot">
     <xacro:include filename ="robot_core.xacro" />
+    <xacro:include filename ="gazebo_control.xacro" />
 </robot>

File: description/robot_core.xacro (robot description, xacro)
@@ -42,4 +42,7 @@
         </xacro:inertial_box>
     </link>
+    <gazebo reference="chassis">
+        <material>Gazebo/White</material>
+    </gazebo>
 <!--Left WHELL-->
     <joint name="left_wheel_joint" type="continuous">
@@ -66,4 +69,7 @@
         </xacro:inertial_cylinder>
     </link>
+    <gazebo reference="left_wheel">
+        <material>Gazebo/Blue</material>
+    </gazebo>
 <!--Right WHELL-->
     <joint name="right_wheel_joint" type="continuous">
@@ -90,11 +96,14 @@
         </xacro:inertial_cylinder>
     </link>
-<!--Castor WHELL-->
-    <joint name="castor_wheel" type="fixed">
+    <gazebo reference="right_wheel">
+        <material>Gazebo/Blue</material>
+    </gazebo>
+<!--Caster WHELL-->
+    <joint name="caster_wheel" type="fixed">
         <parent link="chassis"/>
-        <child link="castor_wheel"/>
+        <child link="caster_wheel"/>
         <origin xyz ="0.24 0 0"/>
     </joint>
-    <link name="castor_wheel">
+    <link name="caster_wheel">
         <visual>
            <geometry>
@@ -113,3 +122,8 @@
         </xacro:inertial_sphere>
     </link>
+    <gazebo reference="caster_wheel">
+        <material>Gazebo/Black</material>
+        <mu1 value="0.001"/>
+        <mu2 value="0.001"/>
+    </gazebo>
 </robot>
